Commit message: TCG not working but let's try and get this packaged up

File: data/urdf/sam_auv.urdf.xacro (robot description, xacro)
@@ -11,4 +11,14 @@
   <link name="$(arg robot_namespace)/thruster_link">
   </link>
+  <link name="$(arg robot_namespace)/battery_link">
+  </link>
+  <link name="$(arg robot_namespace)/tcg1_link">
+  </link>
+  <link name="$(arg robot_namespace)/tcg2_link">
+  </link>
+  <!--
+  <link name="$(arg robot_namespace)/vbs_link">
+  </link>
+  -->
   <joint name="$(arg robot_namespace)/thruster_offset" type="fixed">
     <parent link="$(arg robot_namespace)/base_link"/>
@@ -30,3 +40,33 @@
     <limit lower="-0.3" upper="0.3" velocity="0.2" effort="1.0"/>
   </joint>
+  <joint name="$(arg robot_namespace)/lcg_joint" type="prismatic">
+    <parent link="$(arg robot_namespace)/base_link"/>
+    <child link="$(arg robot_namespace)/battery_link"/>
+    <origin rpy="0.0 0.0 0.0" xyz="-0.37 0.0 0.0"/>
+    <axis xyz="1 0 0"/>
+    <limit lower="-0.01" upper="0.01" velocity="0.2" effort="1.0"/>
+  </joint>
+  <!--
+  <joint name="$(arg robot_namespace)/vbs_joint_virt" type="prismatic">
+    <parent link="$(arg robot_namespace)/base_link"/>
+    <child link="$(arg robot_namespace)/vbs_link"/>
+    <origin rpy="0.0 0.0 0.0" xyz="0.0 0.0 0.0"/>
+    <axis xyz="1 0 0"/>
+    <limit lower="0.0" upper="2.0" velocity="0.2" effort="1.0"/>
+  </joint>
+  -->
+  <joint name="$(arg robot_namespace)/tcg_joint1" type="revolute">
+    <parent link="$(arg robot_namespace)/base_link"/>
+    <child link="$(arg robot_namespace)/tcg1_link"/>
+    <origin rpy="0.0 0.0 0.0" xyz="-0.47 0.0 0.0"/>
+    <axis xyz="1 0 0"/>
+    <limit lower="-1.6" upper="1.6" velocity="0.2" effort="1.0"/>
+  </joint>
+  <joint name="$(arg robot_namespace)/tcg_joint2" type="revolute">
+    <parent link="$(arg robot_namespace)/base_link"/>
+    <child link="$(arg robot_namespace)/tcg2_link"/>
+    <origin rpy="0.0 0.0 0.0" xyz="-0.49 0.0 0.0"/>
+    <axis xyz="1 0 0"/>
+    <limit lower="-1.6" upper="1.6" velocity="0.2" effort="1.0"/>
+  </joint>
 </robot>

Commit message: TCG not working but let's try and get this packaged up

File: data/urdf/sam_auv.urdf.xacro (robot description, xacro)
@@ -17,8 +17,4 @@
   <link name="$(arg robot_namespace)/tcg2_link">
   </link>
-  <!--
-  <link name="$(arg robot_namespace)/vbs_link">
-  </link>
-  -->
   <joint name="$(arg robot_namespace)/thruster_offset" type="fixed">
     <parent link="$(arg robot_namespace)/base_link"/>
@@ -47,13 +43,4 @@
     <limit lower="-0.01" upper="0.01" velocity="0.2" effort="1.0"/>
   </joint>
-  <!--
-  <joint name="$(arg robot_namespace)/vbs_joint_virt" type="prismatic">
-    <parent link="$(arg robot_namespace)/base_link"/>
-    <child link="$(arg robot_namespace)/vbs_link"/>
-    <origin rpy="0.0 0.0 0.0" xyz="0.0 0.0 0.0"/>
-    <axis xyz="1 0 0"/>
-    <limit lower="0.0" upper="2.0" velocity="0.2" effort="1.0"/>
-  </joint>
-  -->
   <joint name="$(arg robot_namespace)/tcg_joint1" type="revolute">
     <parent link="$(arg robot_namespace)/base_link"/>

Commit message: Added multibeam link

File: data/urdf/sam_auv.urdf.xacro (robot description, xacro)
@@ -17,4 +17,11 @@
   <link name="$(arg robot_namespace)/tcg2_link">
   </link>
+  <link name="$(arg robot_namespace)/multibeam_down_link">
+  </link>
+  <joint name="$(arg robot_namespace)/mutlibeam_down_joint" type="fixed">
+    <parent link="$(arg robot_namespace)/base_link"/>
+    <child link="$(arg robot_namespace)/multibeam_down_link"/>
+    <origin rpy="1.5707 0.0 -1.5707" xyz="1.20 0.0 -0.07"/>
+  </joint>
   <joint name="$(arg robot_namespace)/thruster_offset" type="fixed">
     <parent link="$(arg robot_namespace)/base_link"/>

Commit message: Changed the frames in stonefish to be the same as in ros

File: data/urdf/sam_auv.urdf.xacro (robot description, xacro)
@@ -5,7 +5,5 @@
   <link name="$(arg robot_namespace)/base_link">
   </link>
-  <link name="$(arg robot_namespace)/thruster_fixture">
-  </link>
-  <link name="$(arg robot_namespace)/thruster_yaw_fixture">
+  <link name="$(arg robot_namespace)/thruster_yaw_link">
   </link>
   <link name="$(arg robot_namespace)/thruster_link">
@@ -19,32 +17,76 @@
   <link name="$(arg robot_namespace)/multibeam_down_link">
   </link>
-  <joint name="$(arg robot_namespace)/mutlibeam_down_joint" type="fixed">
+  <link name="$(arg robot_namespace)/pressure_link">
+  </link>
+  <link name="$(arg robot_namespace)/dvl_link">
+  </link>
+  <link name="$(arg robot_namespace)/imu_link">
+  </link>
+  <link name="$(arg robot_namespace)/gps_link">
+  </link>
+  <link name="$(arg robot_namespace)/camera_down_link">
+  </link>
+  <link name="$(arg robot_namespace)/camera_front_right_link">
+  </link>
+  <link name="$(arg robot_namespace)/camera_front_left_link">
+  </link>
+  <joint name="$(arg robot_namespace)/multibeam_down_joint" type="fixed">
     <parent link="$(arg robot_namespace)/base_link"/>
     <child link="$(arg robot_namespace)/multibeam_down_link"/>
-    <origin rpy="1.5707 0.0 -1.5707" xyz="1.20 0.0 -0.07"/>
+    <origin rpy="0.0 1.5707 0.0" xyz="1.20 0.0 -0.07"/>
   </joint>
-  <joint name="$(arg robot_namespace)/thruster_offset" type="fixed">
+  <joint name="$(arg robot_namespace)/pressure_joint" type="fixed">
     <parent link="$(arg robot_namespace)/base_link"/>
-    <child link="$(arg robot_namespace)/thruster_fixture"/>
-    <origin rpy="0.0 0.0 0.0" xyz="-0.79 0 0"/>
+    <child link="$(arg robot_namespace)/pressure_link"/>
+    <origin rpy="0.0 0.0 0.0" xyz="0.3 0.0 0.07"/>
   </joint>
-  <joint name="$(arg robot_namespace)/joint1" type="revolute">
-    <parent link="$(arg robot_namespace)/thruster_fixture"/>
-    <child link="$(arg robot_namespace)/thruster_yaw_fixture"/>
+  <joint name="$(arg robot_namespace)/dvl_joint" type="fixed">
+    <parent link="$(arg robot_namespace)/base_link"/>
+    <child link="$(arg robot_namespace)/dvl_link"/>
+    <origin rpy="0.0 0.0 0.0" xyz="1.25 0.0 -0.07"/>
+  </joint>
+  <joint name="$(arg robot_namespace)/imu_joint" type="fixed">
+    <parent link="$(arg robot_namespace)/base_link"/>
+    <child link="$(arg robot_namespace)/imu_link"/>
+    <origin rpy="0.0 0.0 0.0" xyz="0.9 0.0 0.0"/>
+  </joint>
+  <joint name="$(arg robot_namespace)/gps_joint" type="fixed">
+    <parent link="$(arg robot_namespace)/base_link"/>
+    <child link="$(arg robot_namespace)/gps_link"/>
+    <origin rpy="0.0 1.5707 0.0" xyz="1.2 0.0 0.08"/>
+  </joint>
+  <joint name="$(arg robot_namespace)/camera_down_joint" type="fixed">
+    <parent link="$(arg robot_namespace)/base_link"/>
+    <child link="$(arg robot_namespace)/camera_down_link"/>
+    <origin rpy="3.1416 0.0 -1.5707" xyz="1.15 0.0 -0.07"/>
+  </joint>
+  <joint name="$(arg robot_namespace)/camera_front_right_joint" type="fixed">
+    <parent link="$(arg robot_namespace)/base_link"/>
+    <child link="$(arg robot_namespace)/camera_front_right_link"/>
+    <origin rpy="1.3 3.1416 2.3416" xyz="1.32 0.05 0.005"/>
+  </joint>
+  <joint name="$(arg robot_namespace)/camera_front_left_joint" type="fixed">
+    <parent link="$(arg robot_namespace)/base_link"/>
+    <child link="$(arg robot_namespace)/camera_front_left_link"/>
+    <origin rpy="1.3 3.1416 0.8" xyz="1.32 -0.05 0.005"/>
+  </joint>
+  <joint name="$(arg robot_namespace)/thruster_yaw_joint" type="revolute">
+    <parent link="$(arg robot_namespace)/base_link"/>
+    <child link="$(arg robot_namespace)/thruster_yaw_link"/>
     <origin rpy="0.0 0.0 0.0" xyz="0.0 0.0 0.0"/>
     <axis xyz="0 0 1"/>
-    <limit lower="-0.3" upper="0.3" velocity="0.2" effort="1.0"/>
+    <limit lower="-0.2" upper="0.2" velocity="0.2" effort="1.0"/>
   </joint>
-  <joint name="$(arg robot_namespace)/joint2" type="revolute">
-    <parent link="$(arg robot_namespace)/thruster_yaw_fixture"/>
+  <joint name="$(arg robot_namespace)/thruster_pitch_joint" type="revolute">
+    <parent link="$(arg robot_namespace)/thruster_yaw_link"/>
     <child link="$(arg robot_namespace)/thruster_link"/>
-    <origin rpy="0.0 0.0 0.0" xyz="0.1065 0.0 0.0"/>
+    <origin rpy="0.0 0.0 0.0" xyz="0.0 0.0 0.0"/>
     <axis xyz="0 1 0"/>
-    <limit lower="-0.3" upper="0.3" velocity="0.2" effort="1.0"/>
+    <limit lower="-0.2" upper="0.2" velocity="0.2" effort="1.0"/>
   </joint>
   <joint name="$(arg robot_namespace)/lcg_joint" type="prismatic">
     <parent link="$(arg robot_namespace)/base_link"/>
     <child link="$(arg robot_namespace)/battery_link"/>
-    <origin rpy="0.0 0.0 0.0" xyz="-0.37 0.0 0.0"/>
+    <origin rpy="0.0 0.0 0.0" xyz="0.76 0.0 0.0"/>
     <axis xyz="1 0 0"/>
     <limit lower="-0.01" upper="0.01" velocity="0.2" effort="1.0"/>
@@ -53,5 +95,5 @@
     <parent link="$(arg robot_namespace)/base_link"/>
     <child link="$(arg robot_namespace)/tcg1_link"/>
-    <origin rpy="0.0 0.0 0.0" xyz="-0.47 0.0 0.0"/>
+    <origin rpy="0.0 0.0 0.0" xyz="0.48 0.0 0.0"/>
     <axis xyz="1 0 0"/>
     <limit lower="-1.6" upper="1.6" velocity="0.2" effort="1.0"/>
@@ -60,5 +102,5 @@
     <parent link="$(arg robot_namespace)/base_link"/>
     <child link="$(arg robot_namespace)/tcg2_link"/>
-    <origin rpy="0.0 0.0 0.0" xyz="-0.49 0.0 0.0"/>
+    <origin rpy="0.0 0.0 0.0" xyz="0.46 0.0 0.0"/>
     <axis xyz="1 0 0"/>
     <limit lower="-1.6" upper="1.6" velocity="0.2" effort="1.0"/>
